Commit message: include reverse urdf

File: reverse.urdf (robot description, URDF)
Before this commit: robot stewart_platform, 4 links, 3 joints
Links:
- added link arm1, mass 0.03; collision mesh filename=meshes/arm.stl scale=0.001 0.001 0.001; visual mesh filename=meshes/arm.stl scale=0.001 0.001 0.001
- added link arm2, mass 0.025; collision mesh filename=meshes/arm.stl scale=0.001 0.001 0.001; visual mesh filename=meshes/arm.stl scale=0.001 0.001 0.001
- added link arm3, mass 0.025; collision mesh filename=meshes/arm.stl scale=0.001 0.001 0.001; visual mesh filename=meshes/arm.stl scale=0.001 0.001 0.001
- added link base_link
- added link dot1, mass 0.025; collision mesh filename=meshes/dot.stl scale=0.001 0.001 0.001; visual mesh filename=meshes/dot.stl scale=0.001 0.001 0.001
- added link dot1_base, mass 0.025; visual box size=0.005 0.005 0.015
- added link dot2, mass 0.025; collision mesh filename=meshes/dot.stl scale=0.001 0.001 0.001; visual mesh filename=meshes/dot.stl scale=0.001 0.001 0.001
- added link dot2_base, mass 0.025; visual box size=0.005 0.005 0.015
- added link dot3, mass 0.025; collision mesh filename=meshes/dot.stl scale=0.001 0.001 0.001; visual mesh filename=meshes/dot.stl scale=0.001 0.001 0.001
- added link dot3_base, mass 0.025; visual box size=0.005 0.005 0.015
Joints:
- added joint base_to_dot1_base: type fixed, parent base_link, child dot1_base, origin xyz=X1 Y1 Z1 rpy=0 0 0
- added joint base_to_dot2_base: type fixed, parent base_link, child dot2_base, origin xyz=X2 Y2 Z2 rpy=0 0 0
- added joint base_to_dot3_base: type fixed, parent base_link, child dot3_base, origin xyz=X3 Y3 Z3 rpy=0 0 0
- added joint joint_arm1_to_dot1: type revolute, parent arm1, child dot1, origin xyz=-0.041 0.0068 -0.07 rpy=0 0 0, axis 0 1 0, limit lower=-1.57 upper=1.57 effort=1 velocity=1
- added joint joint_arm2_to_dot2: type revolute, parent arm2, child dot2, origin xyz=-0.041 0.0068 -0.07 rpy=0 0 0, axis 0 1 0, limit lower=-1.57 upper=1.57 effort=1 velocity=1
- added joint joint_arm3_to_dot3: type revolute, parent arm3, child dot3, origin xyz=-0.041 0.0068 -0.07 rpy=0 0 0, axis 0 1 0, limit lower=-1.57 upper=1.57 effort=1 velocity=1
- added joint joint_dot1_dot1_base: type fixed, parent dot1, child dot1_base, origin xyz=0.010 -0.0088 0 rpy=0 0 0
- added joint joint_dot2_dot2_base: type fixed, parent dot2, child dot2_base, origin xyz=0.010 -0.0088 0 rpy=0 0 0
- added joint joint_dot3_dot3_base: type fixed, parent dot3, child dot3_base, origin xyz=0.010 -0.0088 0 rpy=0 0 0
- added joint tip1_to_arm1: type revolute, parent arm1_tip, child arm1, origin xyz=0 0 0 rpy=0 0 0, axis 0 1 0, limit lower=-1.57 upper=1.57 effort=1 velocity=1
- added joint tip2_to_arm2: type revolute, parent arm2_tip, child arm2, origin xyz=0 0 0 rpy=0 0 0, axis 0 1 0, limit lower=-1.57 upper=1.57 effort=1 velocity=1
- added joint tip3_to_arm3: type revolute, parent arm3_tip, child arm3, origin xyz=0 0 0 rpy=0 0 0, axis 0 1 0, limit lower=-1.57 upper=1.57 effort=1 velocity=1
- joint joint_top_to_tip1: axis 0 1 0 -> 1 0 0
