Commit message: add collitions

File: robot.urdf (robot description, URDF)
Before this commit: robot stewart_platform, 14 links, 12 joints
Links:
- removed link top
- link arm1: mass None -> 0.03; geometry collision mesh filename=meshes/arm.stl scale=0.001 0.001 0.001; visual mesh filename=meshes/arm.stl scale=0.001 0.001 0.001
- link arm1_tip: mass None -> 0.01; geometry collision sphere radius=0.005; visual sphere radius=0.005
- link arm2: mass None -> 0.025; geometry collision mesh filename=meshes/arm.stl scale=0.001 0.001 0.001; visual mesh filename=meshes/arm.stl scale=0.001 0.001 0.001
- link arm2_tip: mass None -> 0.005; geometry collision sphere radius=0.005; visual sphere radius=0.005
- link arm3: mass None -> 0.025; geometry collision mesh filename=meshes/arm.stl scale=0.001 0.001 0.001; visual mesh filename=meshes/arm.stl scale=0.001 0.001 0.001
- link arm3_tip: mass None -> 0.005; geometry collision sphere radius=0.005; visual sphere radius=0.005
- link base_link: mass None -> 1.0
- link dot1: mass None -> 0.025; geometry collision mesh filename=meshes/dot.stl scale=0.001 0.001 0.001; visual mesh filename=meshes/dot.stl scale=0.001 0.001 0.001
- link dot1_base: mass None -> 0.025; geometry collision box size=0.005 0.005 0.005; visual box size=0.005 0.005 0.005
- link dot2: mass None -> 0.025; geometry collision mesh filename=meshes/dot.stl scale=0.001 0.001 0.001; visual mesh filename=meshes/dot.stl scale=0.001 0.001 0.001
- link dot2_base: mass None -> 0.000125; geometry collision box size=0.005 0.005 0.005; visual box size=0.005 0.005 0.005
- link dot3: mass None -> 0.025; geometry collision mesh filename=meshes/dot.stl scale=0.001 0.001 0.001; visual mesh filename=meshes/dot.stl scale=0.001 0.001 0.001
- link dot3_base: mass None -> 0.01; geometry collision box size=0.005 0.005 0.005; visual box size=0.005 0.005 0.005

Commit message: fix aligments

File: robot.urdf (robot description, URDF)
Before this commit: robot stewart_platform, 13 links, 12 joints
Joints:
- joint joint_arm1: origin xyz=0.0065 0 -0.006 rpy=0 0 0 -> xyz=-0.012 0 -0.00 rpy=0 0 0
- joint joint_arm1_tip_x: origin xyz=0.018 0 0.075 rpy=0 0 0 -> xyz=0.0415 0.0 0.071 rpy=0 0 0
- joint joint_arm2: origin xyz=0.0065 0 -0.006 rpy=0 0 0 -> xyz=-0.012 0 -0.00 rpy=0 0 0
- joint joint_arm2_tip_x: origin xyz=0.018 0 0.075 rpy=0 0 0 -> xyz=0.0415 0.0 0.071 rpy=0 0 0
- joint joint_arm3: origin xyz=0.0065 0 -0.006 rpy=0 0 0 -> xyz=-0.012 0 -0.00 rpy=0 0 0
- joint joint_arm3_tip_x: origin xyz=0.018 0 0.075 rpy=0 0 0 -> xyz=0.0415 0.0 0.071 rpy=0 0 0

Commit message: update collitions

File: robot.urdf (robot description, URDF)
Before this commit: robot stewart_platform, 13 links, 12 joints
Links:
- link base_link: geometry collision box size=0.25 0.25 0.006; visual box size=0.25 0.25 0.006
- link dot1_base: geometry collision box size=0.005 0.005 0.003; visual box size=0.005 0.005 0.005
- link dot2_base: geometry collision box size=0.005 0.005 0.005; visual box size=0.005 0.005 0.003
- link dot3_base: geometry collision box size=0.005 0.005 0.005; visual box size=0.005 0.005 0.003

Commit message: fix base dots

File: robot.urdf (robot description, URDF)
Before this commit: robot stewart_platform, 13 links, 12 joints
Links:
- link dot1_base: geometry visual box size=0.005 0.005 0.005
- link dot2_base: geometry visual box size=0.005 0.005 0.003
- link dot3_base: geometry visual box size=0.005 0.005 0.003

Commit message: robot setup

File: robot.urdf (robot description, URDF)
Before this commit: robot stewart_platform, 13 links, 12 joints
Links:
- added link top; collision mesh filename=meshes/triangle_filled.stl scale=0.001 0.001 0.001; visual mesh filename=meshes/triangle_filled.stl scale=0.001 0.001 0.001
Joints:
- added joint joint_arm1_tip_y: type revolute, parent arm1_tip, child top, origin xyz=0 0 0 rpy=0 0 0, axis 0 1 0, limit lower=-1.57 upper=1.57 effort=1 velocity=1

Commit message: camera setup

File: robot.urdf (robot description, URDF)
Before this commit: robot stewart_platform, 14 links, 13 joints
Links:
- link top: mass None -> 0.05
